File: ID_BAA_STM32BaseModule_v1/ID_BAA_STM32BaseModule_v1.kicad_pcb (KiCad board)
At the start: 2 copper layers, 17 parts, among them J1 RJ12, J2 RJ12, J3 Connecteur Gauche, J4 Connecteur Droit, J5 Connecteur sortie Gauche, J6 Connecteur sortie Droit, U1 MCP2551-I-P

Commit message: Modif BAA
Parts:
- R1: footprint Resistor_SMD:R_1206_3216Metric_Pad1.42x1.75mm_HandSolder -> Resistor_SMD:R_0805_2012Metric_Pad1.15x1.40mm_HandSolder
- R2, R3, R4, R5: footprint Resistor_SMD:R_1206_3216Metric_Pad1.42x1.75mm_HandSolder -> Resistor_SMD:R_0805_2012Metric
Routing:
- net GND: track 63.1 -> 88.6 mm
- net /RXD_CAN: track 62.8 -> 59.0 mm
- net +5V: track 180.2 -> 179.2 mm
