File: ID_BAA_STM32BaseModule_v1/ID_BAA_STM32BaseModule_v1.sch (KiCad schematic (older format))
At the start: 17 parts, among them J1 RJ12, J2 RJ12, J3 Connecteur Gauche, J4 Connecteur Droit, J5 Connecteur sortie Gauche, J6 Connecteur sortie Droit, U1 MCP2551-I-P

Commit message: Modif BAA
Parts:
- R1: footprint Resistor_SMD:R_1206_3216Metric_Pad1.42x1.75mm_HandSolder -> Resistor_SMD:R_0805_2012Metric_Pad1.15x1.40mm_HandSolder
- R2, R3, R4, R5: footprint Resistor_SMD:R_1206_3216Metric_Pad1.42x1.75mm_HandSolder -> Resistor_SMD:R_0805_2012Metric
Changed lines of the file:
@@
 F 0 "R1" H 5670 4446 50  0000 L CNN
 F 1 "150" H 5670 4355 50  0000 L CNN
-F 2 "Resistor_SMD:R_1206_3216Metric_Pad1.42x1.75mm_HandSolder" V 5530 4400 50  0001 C CNN
+F 2 "Resistor_SMD:R_0805_2012Metric_Pad1.15x1.40mm_HandSolder" V 5530 4400 50  0001 C CNN
 F 3 "~" H 5600 4400 50  0001 C CNN
 	1    5600 4400
@@
 F 0 "R2" H 6970 4446 50  0000 L CNN
 F 1 "150" H 6970 4355 50  0000 L CNN
-F 2 "Resistor_SMD:R_1206_3216Metric_Pad1.42x1.75mm_HandSolder" V 6830 4400 50  0001 C CNN
+F 2 "Resistor_SMD:R_0805_2012Metric" V 6830 4400 50  0001 C CNN
 F 3 "~" H 6900 4400 50  0001 C CNN
 	1    6900 4400
@@
 F 0 "R3" H 8420 4446 50  0000 L CNN
 F 1 "150" H 8420 4355 50  0000 L CNN
-F 2 "Resistor_SMD:R_1206_3216Metric_Pad1.42x1.75mm_HandSolder" V 8280 4400 50  0001 C CNN
+F 2 "Resistor_SMD:R_0805_2012Metric" V 8280 4400 50  0001 C CNN
 F 3 "~" H 8350 4400 50  0001 C CNN
 	1    8350 4400
@@
 F 0 "R4" H 9720 4446 50  0000 L CNN
 F 1 "150" H 9720 4355 50  0000 L CNN
-F 2 "Resistor_SMD:R_1206_3216Metric_Pad1.42x1.75mm_HandSolder" V 9580 4400 50  0001 C CNN
+F 2 "Resistor_SMD:R_0805_2012Metric" V 9580 4400 50  0001 C CNN
 F 3 "~" H 9650 4400 50  0001 C CNN
 	1    9650 4400
@@
 F 0 "R5" H 3420 1846 50  0000 L CNN
 F 1 "10K" H 3420 1755 50  0000 L CNN
-F 2 "Resistor_SMD:R_1206_3216Metric_Pad1.42x1.75mm_HandSolder" V 3280 1800 50  0001 C CNN
+F 2 "Resistor_SMD:R_0805_2012Metric" V 3280 1800 50  0001 C CNN
 F 3 "~" H 3350 1800 50  0001 C CNN
 	1    3350 1800
@@
 $EndComp
 $Comp
-L power:GND #PWR?
+L power:GND #PWR0121
 U 1 1 62574BB8
 P 7850 2050
-F 0 "#PWR?" H 7850 1800 50  0001 C CNN
+F 0 "#PWR0121" H 7850 1800 50  0001 C CNN
 F 1 "GND" V 7855 1922 50  0000 R CNN
 F 2 "" H 7850 2050 50  0001 C CNN
@@
 $EndComp
 $Comp
-L power:GND #PWR?
+L power:GND #PWR0122
 U 1 1 6257523F
 P 7850 2150
-F 0 "#PWR?" H 7850 1900 50  0001 C CNN
+F 0 "#PWR0122" H 7850 1900 50  0001 C CNN
 F 1 "GND" V 7855 2022 50  0000 R CNN
 F 2 "" H 7850 2150 50  0001 C CNN
