File: ID_BAC_Carte_Alimentation/ID_BAC_Carte_Alimentation.kicad_pcb (KiCad board)
At the start: 2 copper layers, 66 x 91.4 mm, 14 parts, among them J1 connector_battery, J2 RJ_can, J3 connector_battery, U1 JCK2012S12, U2 JCK2012S05

Commit message: Carte_alim serigraphy
Other:
- board text added: "Andrea Perez Fernandez 2022 ID Carte : BAC"
Changed lines of the file:
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@@
       (xy 170.18 25.4)
     ) (layer "Edge.Cuts") (width 0.1) (fill none))
+  (gr_text "Andrea Perez Fernandez \n2022\nID Carte : BAC \n" (at 137.668 69.342) (layer "B.SilkS")
+    (effects (font (size 2 2) (thickness 0.15)) (justify mirror))
+  )
   (gr_text "12V" (at 143.256 103.378) (layer "F.SilkS")
     (effects (font (size 1 1) (thickness 0.15)))
